File: pcb/rgb_matrix.kicad_sch (KiCad schematic)
At the start: 10 parts

Commit message: Still tidying pcb design
Parts:
- added C10, C11, C12, C13, C14, C15, C16, C17, C18, C9: 100nF, Capacitor_SMD:C_0402_1005Metric, symbol Device:C
Connections:
- net 3-5V: now also C10.2, C11.2, C12.2, C13.2, C14.2, C15.2, C16.2, C17.2, C18.2, C9.2
- net GND: now also C10.1, C11.1, C12.1, C13.1, C14.1, C15.1, C16.1, C17.1, C18.1, C9.1
Other:
- moved on the sheet: D12, D13, D14, D15

Commit message: Still improving pcb, I learned what a fiducial is today
Parts:
- added C3: 100uf, Capacitor_SMD:CP_Elec_4x5.4, symbol Device:C_Polarized
Connections:
- net GND: now also C3.2
- net 3-5V renamed VSYS
- net VSYS: now also C3.1

Commit message: I think the PCB is almost done for real this time chat. Just gotta add part numbers for the BOM
Parts:
- added Q2: AO3401A, Package_TO_SOT_SMD:SOT-23, symbol Transistor_FET:AO3401A
- added Q3: 2N7002E, Package_TO_SOT_SMD:SOT-23, symbol Transistor_FET:2N7002E
- added R14: 300, Resistor_SMD:R_0603_1608Metric, symbol Device:R
- added R17, R18: 100k, Resistor_SMD:R_0603_1608Metric, symbol Device:R
- C10, C11, C12, C13, C14, C15, C16, C17, C18, C9: value 100nF -> 0.1uf
Connections:
- net Data: now also R14.2; no longer D6.4 (DIN)
- net GND: now also Q3.2 (S), R18.2
- net VSYS: now also Q2.2 (S), R17.1; no longer C10.2, C11.2, C12.2, C13.2, C14.2, C15.2, C16.2, C17.2, C18.2, C3.1, C9.2, D10.1 (VDD), D11.1 (VDD), D12.1 (VDD), D13.1 (VDD), D14.1 (VDD), D15.1 (VDD), D6.1 (VDD), D7.1 (VDD), D8.1 (VDD), D9.1 (VDD)
- new net: C10.2, C11.2, C12.2, C13.2, C14.2, C15.2, C16.2, C17.2, C18.2, C3.1, C9.2, D10.1 (VDD), D11.1 (VDD), D12.1 (VDD), D13.1 (VDD), D14.1 (VDD), D15.1 (VDD), D6.1 (VDD), D7.1 (VDD), D8.1 (VDD), D9.1 (VDD), Q2.3 (D)
- new net: Q2.1 (G), Q3.3 (D), R17.2
- new net: D6.4 (DIN), R14.1
- new net LEDPower: Q3.1 (G), R18.1
Other:
- moved on the sheet: C10, C11, C12, C13, C14, C15, C16, C17, C18, C3, C9, D10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

Commit message: I think the PCB is ready to ship, just gonna tidy up a couple more things
Parts:
- C10, C11, C12, C13, C14, C15, C16, C17, C18, C9: MPN (none) -> GRM155R71H104KE14D; Manufacturer (none) -> Murata Electronics
- C3: footprint Capacitor_SMD:CP_Elec_4x5.4 -> Capacitor_SMD:C_1206_3216Metric; symbol Device:C_Polarized -> Device:C; MPN (none) -> GRM31CR61A107MEA8L; Manufacturer (none) -> Murata
- D10, D11, D12, D13, D14, D15, D6, D7, D8, D9: MPN (none) -> WS2812B; Manufacturer (none) -> Worldsemi
- Q2: MPN (none) -> AO3401A; Manufacturer (none) -> Alpha & Omega Semiconductor Inc.
- Q3: MPN (none) -> 2N7002E-7-F; Manufacturer (none) -> Diodes Incorporated
- R14: MPN (none) -> ERJ-3GEYJ301V; Manufacturer (none) -> Panasonic Industry
- R17, R18: MPN (none) -> CRCW0603100KFKEA; Manufacturer (none) -> Vishay Dale
