File: pcb/st7789-connector.kicad_sch (KiCad schematic)
At the start: 1 part, among them J2 DISPLAY

Commit message: Still improving pcb, I learned what a fiducial is today
Parts:
- added C1: 0.1uf, Capacitor_SMD:C_0402_1005Metric, symbol Device:C
- added Q1: 2N7002E, Package_TO_SOT_SMD:SOT-23, symbol Transistor_FET:2N7002E
- added R10: 20, Resistor_SMD:R_0603_1608Metric, symbol Device:R
- J2: symbol Connector_Generic:Conn_01x12 -> Connector_Generic:Conn_01x13
Connections:
- net VDD is gone; now on net +3.3V: J2.4 (Pin_4)
- net GND: now also J2.MP (Pin_13), C1.1, Q1.2 (S)
- net LEDK: now also Q1.1 (G); no longer J2.2 (Pin_2)
- net LEDA renamed +3.3V
- net +3.3V: now also C1.2
- new net: Q1.3 (D), R10.1
- new net: J2.2 (Pin_2), R10.2

Commit message: I think the PCB is almost done for real this time chat. Just gotta add part numbers for the BOM
Parts:
- J2: value DISPLAY -> FH12-12S-0.5SH
Changed lines of the file:
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@@
+			)
+		)
+		(property "Sim.Device" ""
+			(at 168.91 115.57 0)
+			(hide yes)
+			(show_name no)
+			(do_not_autoplace no)
+			(effects
+				(font
+					(size 1.27 1.27)
+				)
+			)
+		)
+		(property "Sim.Type" ""
+			(at 168.91 115.57 0)
+			(hide yes)
+			(show_name no)
+			(do_not_autoplace no)
+			(effects
+				(font
+					(size 1.27 1.27)
+				)
 			)
 		)
@@
 			)
 		)
-		(property "Value" "DISPLAY"
+		(property "Value" "FH12-12S-0.5SH"
 			(at 138.43 78.74 0)
 			(show_name no)
@@
 			)
 		)
-		(property "Description" "Generic connector, single row, 01x13, script generated (kicad-library-utils/schlib/autogen/connector/)"
+		(property "Description" "ST7789 display FFC, 12-pin, 0.5 mm pitch"
+			(at 138.43 97.79 0)
+			(hide yes)
+			(show_name no)
+			(do_not_autoplace no)
+			(effects
+				(font
+					(size 1.27 1.27)
+				)
+			)
+		)
+		(property "Sim.Device" ""
+			(at 138.43 97.79 0)
+			(hide yes)
+			(show_name no)
+			(do_not_autoplace no)
+			(effects
+				(font
+					(size 1.27 1.27)
+				)
+			)
+		)
+		(property "Sim.Type" ""
 			(at 138.43 97.79 0)
 			(hide yes)
@@
 			)
 		)
+		(property "Sim.Device" ""
+			(at 166.37 101.6 90)
+			(hide yes)
+			(show_name no)
+			(do_not_autoplace no)
+			(effects
+				(font
+					(size 1.27 1.27)
+				)
+			)
+		)
+		(property "Sim.Type" ""
+			(at 166.37 101.6 90)
+			(hide yes)
+			(show_name no)
+			(do_not_autoplace no)
+			(effects
+				(font
+					(size 1.27 1.27)
+				)
+			)
+		)
 		(pin "1"
 		)
@@
 			(hide yes)
 			(show_name no)
+			(do_not_autoplace no)
+			(effects
+				(font
+					(size 1.27 1.27)
+				)
+			)
+		)
+		(property "Sim.Device" ""
+			(at 160.02 110.49 90)
+			(hide yes)
+			(show_name no)
+			(do_not_autoplace no)
+			(effects
+				(font
+					(size 1.27 1.27)
+				)
+			)
+		)
+		(property "Sim.Type" ""
+			(at 160.02 110.49 90)
+			(hide yes)
+			(show_name no)

Commit message: I think the PCB is ready to ship, just gonna tidy up a couple more things
Parts:
- C1: MPN (none) -> GRM155R71H104KE14D; Manufacturer (none) -> Murata Electronics
- J2: value FH12-12S-0.5SH -> FFC2B28-12-G; footprint Connector_FFC-FPC:Hirose_FH12-12S-0.5SH_1x12-1MP_P0.50mm_Horizontal -> FFC2B28-12-G:GCT_FFC2B28-12-G; symbol Connector_Generic:Conn_01x13 -> FFC2B28-12-G:FFC2B28-12-G; Check_prices (none) -> https://www.snapeda.com/parts/FFC2B28-12-G/Global+Connector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; DigiKey_Part_Number (none) -> 2073-FFC2B28-12-GCT-ND; MANUFACTURER (none) -> GCT; MAXIMUM_PACKAGE_HEIGHT (none) -> 1.75mm; MF (none) -> Global Connector Technology; MP (none) -> FFC2B28-12-G; MPN (none) -> FFC2B28-12-G; Manufacturer (none) -> GCT; PARTREV (none) -> A; Package (none) -> None; STANDARD (none) -> Manufacturer Recommendations; SilkLabel (none) -> DISPLAY; SnapEDA_Link (none) -> https://www.snapeda.com/parts/FFC2B28-12-G/Global+Connector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
- Q1: MPN (none) -> 2N7002E-7-F; Manufacturer (none) -> Diodes Incorporated
- R10: MPN (none) -> RMCF0603JT20R0; Manufacturer (none) -> Stackpole Electronics Inc
Connections:
- net GND: now also J2.S1 (SHIELD), J2.S2 (SHIELD); no longer J2.MP (Pin_13)
Other:
- moved on the sheet: J2
