File: pcb/trackball.kicad_sch (KiCad schematic)
At the start: 21 parts, among them SW1 BTN, U1 UP, U2 DWN, U3 LFT, U4 RHT

Commit message: Still improving pcb, I learned what a fiducial is today
Connections:
- net +3v3 renamed +3.3V

Commit message: I think the PCB is almost done for real this time chat. Just gotta add part numbers for the BOM
Parts:
- added C19: 0.1uf, Capacitor_SMD:C_0402_1005Metric, symbol Device:C
- added R19, R20: 4.7k, Resistor_SMD:R_0603_1608Metric, symbol Device:R
- added U5: PCA9633DP1:PCA9633DP1, Package_SO:TSSOP-8_3x3mm_P0.65mm, symbol PCA9633:PCA9633DP1
- C4, C5, C6, C7: footprint Capacitor_SMD:C_01005_0402Metric -> Capacitor_SMD:C_0402_1005Metric
- D1: value BLU -> BLUE
- D3: value GRN -> GREEN
- D4: value WHT -> WHITE
- R5, R6, R7, R8: now not fitted
Connections:
- net BLU is gone; now on net +3.3V: R1.2
- net GRN is gone; now on net +3.3V: R3.2
- net RED is gone; now on net +3.3V: R2.2
- net WHT is gone; now on net +3.3V: R4.2
- net +3.3V: now also C19.2, R19.2, R20.2, U5.8 (VDD)
- net GND: now also C19.1, U5.5 (VSS); no longer D1.1 (K), D2.1 (K), D3.1 (K), D4.1 (K)
- new net: D3.1 (K), U5.4 (LED3)
- new net: D2.1 (K), U5.1 (LED0)
- new net: D4.1 (K), U5.2 (LED1)
- new net: D1.1 (K), U5.3 (LED2)
- new net SCL0: R20.1, U5.6 (SCL)
- new net SDA0: R19.1, U5.7 (SDA)
Other:
- moved on the sheet: D1, D2, D3, D4, R1, R2, R3, R4

Commit message: I think the PCB is ready to ship, just gonna tidy up a couple more things
Parts:
- C19, C4, C5, C6, C7: MPN (none) -> GRM155R71H104KE14D; Manufacturer (none) -> Murata Electronics
- D1: footprint LED_SMD:LED_0201_0603Metric -> LED_SMD:LED_0402_1005Metric; MPN (none) -> APHHS1005QBC/D; Manufacturer (none) -> Kingbright; SilkLabel (none) -> BLUE
- D2: footprint LED_SMD:LED_0201_0603Metric -> LED_SMD:LED_0402_1005Metric; MPN (none) -> APHHS1005SURCK; Manufacturer (none) -> Kingbright; SilkLabel (none) -> RED
- D3: footprint LED_SMD:LED_0201_0603Metric -> LED_SMD:LED_0402_1005Metric; MPN (none) -> APHHS1005ZGC; Manufacturer (none) -> Kingbright; SilkLabel (none) -> GREEN
- D4: footprint LED_SMD:LED_0201_0603Metric -> LED_SMD:LED_0402_1005Metric; MPN (none) -> IN-S42BT5UW; Manufacturer (none) -> Inolux; SilkLabel (none) -> WHITE
- R1, R4: MPN (none) -> RC0201FR-07180RL; Manufacturer (none) -> Yageo
- R19, R20: MPN (none) -> RC0603FR-074K7L; Manufacturer (none) -> Yageo
- R2: value 180 -> 360; MPN (none) -> RC0201FR-07360RL; Manufacturer (none) -> Yageo
- R3: value 180 -> 330; MPN (none) -> RC0201FR-07330RL; Manufacturer (none) -> Yageo
- R5, R6, R7, R8: MPN (none) -> RC0201FR-0710KL; Manufacturer (none) -> Yageo
- SW1: MPN (none) -> TL3315NF100Q; Manufacturer (none) -> E-Switch
- U1: value UP -> TMAG5231C1GQDBZR; MPN (none) -> TMAG5231C1GQDBZR; Manufacturer (none) -> Texas Instruments; SilkLabel (none) -> UP
- U2: value DWN -> TMAG5231C1GQDBZR; MPN (none) -> TMAG5231C1GQDBZR; Manufacturer (none) -> Texas Instruments; SilkLabel (none) -> DOWN
- U3: value LFT -> TMAG5231C1GQDBZR; MPN (none) -> TMAG5231C1GQDBZR; Manufacturer (none) -> Texas Instruments; SilkLabel (none) -> LEFT
- U4: value RHT -> TMAG5231C1GQDBZR; MPN (none) -> TMAG5231C1GQDBZR; Manufacturer (none) -> Texas Instruments; SilkLabel (none) -> RIGHT
- U5: value PCA9633DP1:PCA9633DP1 -> PCA9633DP1; MPN (none) -> PCA9633DP1,118; Manufacturer (none) -> NXP USA Inc.
Connections:
- net +3.3V: no longer R1.2, R2.2, R3.2, R4.2
- net SCL0 renamed SCL
- net SDA0 renamed SDA
- new net VSYS: R1.2, R2.2, R3.2, R4.2
